File: gem-demo-board.sch (KiCad schematic (older format))
At the start: 147 parts, among them J1 3220-10-0100-00, J10 0473460001, J2 DF13A-2P-1.25H, J3 3220-10-0100-00, J4 2x20_Header_Female, J5 0473460001, J6 556500488, J7 556500488, J8 WE_686115148922_FLIPPED, J9 WE_686115148922_FLIPPED, U1 MCP1700T-3302E_TT, U2 NTS0104BQ, U3 NTS0104BQ, U4 NTS0104BQ, U5 93LC56CT-IMC, U6 FT4232HQ, U7 NTB0104BQ, U8 NTB0104BQ, Y1 ASFLMB-12.000MHZ-LC-T

Commit message: Moved JTAG connector
Parts:
- R44, R45, R46, R47, R50, R51, R52, R53, R54, R55, R56, R57: DNP (none) -> 1
- U5: MPN (none) -> 93LC56CT-I/MC; Manufactuer (none) -> Microchip
Changed lines of the file:
@@
 encoding utf-8
 Sheet 1 1
-Title "GEM Demo Board"
+Title "GEM1 Demo Board"
 Date ""
 Rev "1.1"
-Comp "Antmicro"
-Comment1 "www.antmicro.com"
-Comment2 ""
+Comp ""
+Comment1 "Antmicro Ltd."
+Comment2 "www.antmicro.com"
 Comment3 ""
 Comment4 ""
@@
 F 2 "gem-demo-board-footprints:DFN-8_2x3mm" H 1450 9600 50  0001 C CNN
 F 3 "http://ww1.microchip.com/downloads/en/DeviceDoc/20001749K.pdf" H 1850 9450 50  0001 C CNN
+F 4 "93LC56CT-I/MC" H 1850 9450 50  0001 C CNN "MPN"
+F 5 "Microchip" H 1850 9450 50  0001 C CNN "Manufactuer"
 	1    1850 9450
 	1    0    0    -1
@@
 F 5 "ERJ2GE0R00X" H 11000 4550 60  0001 L CNN "MPN"
 F 6 "0R" H 11000 4300 50  0000 C CNN "Val"
+F 7 "1" H 10800 4250 50  0001 C CNN "DNP"
 	1    10800 4250
 	1    0    0    -1
@@
 F 5 "ERJ2GE0R00X" H 11000 4650 60  0001 L CNN "MPN"
 F 6 "0R" H 11000 4400 50  0000 C CNN "Val"
+F 7 "1" H 10800 4350 50  0001 C CNN "DNP"
 	1    10800 4350
 	1    0    0    -1
@@
 F 5 "ERJ2GE0R00X" H 11000 4750 60  0001 L CNN "MPN"
 F 6 "0R" H 11000 4500 50  0000 C CNN "Val"
+F 7 "1" H 10800 4450 50  0001 C CNN "DNP"
 	1    10800 4450
 	1    0    0    -1
@@
 F 5 "ERJ2GE0R00X" H 11000 4850 60  0001 L CNN "MPN"
 F 6 "0R" H 11000 4600 50  0000 C CNN "Val"
+F 7 "1" H 10800 4550 50  0001 C CNN "DNP"
 	1    10800 4550
 	1    0    0    -1
@@
 F 5 "ERJ2GE0R00X" H 12500 6100 60  0001 L CNN "MPN"
 F 6 "0R" H 12500 5850 50  0000 C CNN "Val"
+F 7 "1" H 12300 5800 50  0001 C CNN "DNP"
 	1    12300 5800
 	1    0    0    -1
@@
 F 5 "ERJ2GE0R00X" H 12500 6250 60  0001 L CNN "MPN"
 F 6 "0R" H 12500 6000 50  0000 C CNN "Val"
+F 7 "1" H 12300 5950 50  0001 C CNN "DNP"
 	1    12300 5950
 	1    0    0    -1
@@
 F 5 "ERJ2GE0R00X" H 12500 6500 60  0001 L CNN "MPN"
 F 6 "0R" H 12500 6250 50  0000 C CNN "Val"
+F 7 "1" H 12300 6200 50  0001 C CNN "DNP"
 	1    12300 6200
 	1    0    0    -1
@@
 F 5 "ERJ2GE0R00X" H 12500 6650 60  0001 L CNN "MPN"
 F 6 "0R" H 12500 6400 50  0000 C CNN "Val"
+F 7 "1" H 12300 6350 50  0001 C CNN "DNP"
 	1    12300 6350
 	1    0    0    -1
@@
 F 5 "ERJ2GE0R00X" H 12500 6950 60  0001 L CNN "MPN"
 F 6 "0R" H 12500 6700 50  0000 C CNN "Val"
+F 7 "1" H 12300 6650 50  0001 C CNN "DNP"
 	1    12300 6650
 	1    0    0    -1
@@
 F 5 "ERJ2GE0R00X" H 12500 7100 60  0001 L CNN "MPN"
 F 6 "0R" H 12500 6850 50  0000 C CNN "Val"
+F 7 "1" H 12300 6800 50  0001 C CNN "DNP"
 	1    12300 6800
 	1    0    0    -1
@@
 F 5 "ERJ2GE0R00X" H 12500 5700 60  0001 L CNN "MPN"
 F 6 "0R" H 12500 5450 50  0000 C CNN "Val"
+F 7 "1" H 12300 5400 50  0001 C CNN "DNP"
 	1    12300 5400
 	1    0    0    -1
@@
 F 5 "ERJ2GE0R00X" H 12500 5850 60  0001 L CNN "MPN"
 F 6 "0R" H 12500 5600 50  0000 C CNN "Val"
+F 7 "1" H 12300 5550 50  0001 C CNN "DNP"
 	1    12300 5550
 	1    0    0    -1

Commit message: Fixed MPN for 12Mhz oscillator
Parts:
- Y1: MPN 7C-24.000MBB-T -> ASFLMB-12.000MHZ-LC-T
Changed lines of the file:
@@
 F 2 "gem-demo-board-footprints:ASFLMB" H 2750 10400 50  0001 C CNN
 F 3 "" H 2600 11200 50  0001 C CNN
-F 4 "7C-24.000MBB-T" H 2550 11000 50  0001 C CNN "MPN"
+F 4 "ASFLMB-12.000MHZ-LC-T" H 2550 11000 50  0001 C CNN "MPN"
 F 5 "TXC" H 2500 11100 50  0001 C CNN "Manufacturer"
 	1    2500 10700
